Commit message: new gx10 and ex12

File: retargeting/urdf/ex12/urdf/ex12.urdf (robot description, URDF)
Before this commit: robot ex12, 16 links, 15 joints
Links:
- link Link1: mass 0.0217307435979103 -> 0.0224844737579923
- link Link10: mass 0.0265839433569182 -> 0.0192719642321749
- link Link11: mass 0.0230133561838601 -> 0.0213744172444923
- link Link2: mass 0.0220862243589131 -> 0.0238979446909479
- link Link3: mass 0.0195941447971888 -> 0.021951062818985
- link Link5: mass 0.0178831940703488 -> 0.017883193977129
- link Link6: mass 0.0265839433569186 -> 0.019271964232175
- link Link7: mass 0.0230133561838601 -> 0.0213744172444923
- link Link8: mass 0.00344356132156392 -> 0.00344356132156391
- link Link9: mass 0.0178831940205361 -> 0.0178831939273071
- link base_link: mass 0.100282584501496 -> 0.104869110532873
Joints:
- joint joint1: limit lower=-0.5236 upper=1.5708 effort=10 velocity=3.1 -> lower=-3.1415 upper=3.1415 effort=1 velocity=10; origin xyz=0.0726385389055488 -0.00636396103067888 0.0098 rpy=-1.5707963267949 0 -0.785398163397448 -> xyz=0.0751385389055488 -0.00636396103067887 0.0048 rpy=-1.5707963267949 0 -0.785398163397448
- joint joint10: axis 0 0 -1 -> 0 0 1; limit lower=-3.14 upper=3.14 effort=10 velocity=3.1 -> lower=-3.1415 upper=3.1415 effort=1 velocity=10; origin xyz=0 0 -0.013 rpy=1.5707963267949 -0.192944037979531 0 -> xyz=0 0 -0.013 rpy=1.5707963267949 0 0
- joint joint11: axis 0 0 -1 -> 0 0 1; limit lower=-3.14 upper=3.14 effort=10 velocity=3.1 -> lower=-3.1415 upper=3.1415 effort=1 velocity=10; origin xyz=0.0850000000000001 0 0 rpy=0 0 -1.90426963990731 -> xyz=0.0780000000000002 0 0 rpy=0 0 -0.333473313112389
- joint joint12: limit lower=-3.14 upper=3.14 effort=10 velocity=3.1 -> lower=-3.1415 upper=3.1415 effort=1 velocity=10; origin xyz=0.0727581521785941 0 0 rpy=3.14159265358979 0 -0.383069500465414 -> xyz=0.0727581521785949 0 0 rpy=0 0 -0.713724238084212
- joint joint13: limit (none) -> lower=-3.1415 upper=3.1415 effort=1 velocity=10; origin xyz=0 -0.0405 0 rpy=1.5707963267949 0 0 -> xyz=0 -0.0404999999999942 -0.00600000000019235 rpy=3.14159265358979 -0.26179938779915 -1.57079632679494
- joint joint14: origin xyz=0.0405 0 0 rpy=3.14159265358979 0 -1.5707963267949 -> xyz=0.0405 0 0 rpy=0 0 1.0471975511966
- joint joint15: origin xyz=0.0405 0 0 rpy=3.1416 0 -1.5708 -> xyz=0.040224 0 0.00020018 rpy=0 0 1.0472
- joint joint2: limit lower=-3.14 upper=3.14 effort=10 velocity=3.1 -> lower=-3.1415 upper=3.1415 effort=1 velocity=10; origin xyz=0 -0.0142 0.0455 rpy=1.5707963267949 -0.785398163397449 -3.14159265358979 -> xyz=0 -0.0192 0.0555 rpy=-1.63723082087563 -1.57079630572147 0.0664344940807344
- joint joint3: limit lower=-3.14 upper=3.14 effort=10 velocity=3.1 -> lower=-3.1415 upper=3.1415 effort=1 velocity=10; origin xyz=0.0555 0 0 rpy=0 0 0 -> xyz=0.085 0 0 rpy=0 0 2.94060183304342
- joint joint4: axis 0 0 -1 -> 0 0 1; limit lower=-3.14 upper=3.14 effort=10 velocity=3.1 -> lower=-3.1415 upper=3.1415 effort=1 velocity=10; origin xyz=0.0445 0 0 rpy=0 0 0 -> xyz=-0.0766132032286162 0.00563403969797617 0 rpy=2.41700305744513 1.5707963267949 0
- joint joint5: axis 0 0 -1 -> 0 0 1; limit lower=-3.14 upper=3.14 effort=10 velocity=3.1 -> lower=-3.1415 upper=3.1415 effort=1 velocity=10; origin xyz=0.015 0.076293277315303 -0.0509166604983955 rpy=0 0.5235987755983 1.5707963267949 -> xyz=0.0175 0.0814594408408979 -0.034 rpy=0 0 1.5707963267949
- joint joint6: limit lower=-3.14 upper=3.14 effort=10 velocity=3.1 -> lower=-3.1415 upper=3.1415 effort=1 velocity=10; origin xyz=0 0 0.013 rpy=-1.5707963267949 0.192944037979531 0 -> xyz=0 0 0.013 rpy=-1.5707963267949 0 0
- joint joint7: limit lower=-3.14 upper=3.14 effort=10 velocity=3.1 -> lower=-3.1415 upper=3.1415 effort=1 velocity=10; origin xyz=0.0850000000000002 0 0 rpy=0 0 -1.90426963990731 -> xyz=0.0779999999999999 0 0 rpy=0 0 -0.333473313112389
- joint joint8: axis 0 0 1 -> 0 0 -1; limit lower=-3.14 upper=3.14 effort=10 velocity=3.1 -> lower=-3.1415 upper=3.1415 effort=1 velocity=10; origin xyz=0.0727581521785944 0 0 rpy=3.14159265358979 0 -0.383069500465415 -> xyz=0.0727581521785942 0 0 rpy=0 0 -0.713724238084215
- joint joint9: axis 0 0 1 -> 0 0 -1; limit lower=-3.14 upper=3.14 effort=0 velocity=0 -> lower=-3.1415 upper=3.1415 effort=1 velocity=10; origin xyz=-0.015 0.076293277315303 -0.0509166604983955 rpy=-3.14159265358979 0.5235987755983 1.5707963267949 -> xyz=-0.0175 0.0814594408408979 -0.034 rpy=3.14159265358979 0 1.5707963267949

File: retargeting/urdf/gx10/urdf/gx10.urdf (robot description, URDF)
Before this commit: robot gx11, 15 links, 14 joints
Links:
- removed link Link14
- link Link1: mass 0.0204594242505954 -> 0.0231992249064679
- link Link10: mass 0.0222688407505351 -> 0.00125017090070062
- link Link11: mass 0.00125017090070063 -> 0.016424831381844
- link Link12: mass 0.0164248371643224 -> 0.0164248382176841
- link Link13: mass 0.016424837165235 -> 0.0164248317291125
- link Link2: mass 0.0220862252142514 -> 0.0089743671891579
- link Link3: mass 0.00125017090070063 -> 0.0348712226438575
- link Link4: mass 0.0259800201624105 -> 0.00125017090070062
- link Link5: mass 0.0176678393043425 -> 0.00521913649462284
- link Link6: mass 0.0222688407504672 -> 0.0348416546367208
- link Link8: mass 0.0259800201624256 -> 0.00521913649462284
- link Link9: mass 0.0176678393044255 -> 0.0347918481270268
- link base_link: mass 0.160797512292559 -> 0.135870626687155
Joints:
- removed joint joint14
- joint joint1: limit lower=0 upper=2.1 effort=10 velocity=6.2 -> lower=-1 upper=1 effort=5 velocity=3.2; origin xyz=0.0309007440278484 0.0305 0.0058732274974783 rpy=1.5707963267949 0 0 -> xyz=0.0284999999999998 0.0222000000000001 0.0147407332682075 rpy=0 0 0
- joint joint10: axis 0 0 1 -> 0 0 -1; limit lower=-0.506 upper=1.885 effort=10 velocity=6.2 -> lower=-1 upper=1 effort=5 velocity=3.2; origin xyz=0 0 0.013 rpy=1.5708 0 0 -> xyz=0.0489999999999996 0 0 rpy=0 0 0
- joint joint11: axis 0 0 -1 -> 0 0 0; limit lower=-0.366 upper=2.042 effort=10 velocity=6.2 -> (none); origin xyz=0.0359999999999999 0 0 rpy=-3.14159265358979 0 0 -> xyz=0.0599999999999635 -0.00241845943756577 0 rpy=0 1.5707963267949 0; parent Link10 -> Link4; type revolute -> fixed
- joint joint12: limit lower=-1 upper=1 effort=0 velocity=0 -> (none); origin xyz=0.0570187350990352 0.00231569753250521 8.14092925386471E-05 rpy=0 1.5707963267949 0 -> xyz=0.0600000000000002 0.00241854395832904 0 rpy=0 1.5707963267949 0; parent Link3 -> Link7
- joint joint13: origin xyz=0.0570187350990352 -0.00231569753250514 -8.14092925387963E-05 rpy=0 1.5707963267949 0 -> xyz=0.06 -0.0024185 0 rpy=0 -1.5708 3.141593; parent Link7 -> Link10
- joint joint2: axis 0 0 1 -> 0 0 -1; limit lower=-0.25 upper=1.7 effort=10 velocity=6.2 -> lower=-1 upper=1 effort=5 velocity=3.2; origin xyz=0.0344999999999999 0 0.013 rpy=-1.5707963267949 0 0 -> xyz=0.0149999999999997 0 0.017 rpy=-1.5707963267949 0 0
- joint joint3: axis 0 0 1 -> 0 0 -1; limit lower=-0.25 upper=1.7 effort=10 velocity=6.2 -> lower=-1 upper=1 effort=5 velocity=3.2; origin xyz=0.0555000000000001 0 0 rpy=0 0 0 -> xyz=0.035624993619291 -0.00320000000000058 0.000118338320757781 rpy=1.5707963267949 0 0
- joint joint4: limit lower=-0.3 upper=1.6 effort=10 velocity=6.2 -> lower=-1 upper=1 effort=5 velocity=3.2; origin xyz=0.029 0.096 0.00806475912646926 rpy=1.5707963267949 0 1.5707963267949 -> xyz=0.0489999999999997 0 0 rpy=0 0 0; parent base_link -> Link3
- joint joint5: limit lower=-0.6 upper=0.6 effort=10 velocity=6.2 -> lower=-1 upper=1 effort=5 velocity=3.2; origin xyz=0.0515 -0.0119999999999991 0 rpy=-1.5707963267949 0 0 -> xyz=0.0285 0.0765 0.000240733268207483 rpy=0 0 1.5707963267949; parent Link4 -> base_link
- joint joint6: limit lower=-0.506 upper=1.885 effort=10 velocity=6.2 -> lower=-1 upper=1 effort=5 velocity=3.2; origin xyz=0 0 0.013 rpy=1.5707963267949 0 0 -> xyz=0.0300000000000001 0 0 rpy=-1.5707963267949 0 0
- joint joint7: limit lower=-0.366 upper=2.042 effort=10 velocity=6.2 -> lower=-1 upper=1 effort=5 velocity=3.2; origin xyz=0.036 0 0 rpy=3.14159265358979 0 0 -> xyz=0.0489999999999997 0 0 rpy=0 0 0
- joint joint8: axis 0 0 1 -> 0 0 -1; limit lower=-0.314 upper=2.23 effort=10 velocity=6.2 -> lower=-1 upper=1 effort=5 velocity=3.2; origin xyz=-0.0289999999999999 0.096 0.00806475912646949 rpy=1.5707963267949 0 1.5707963267949 -> xyz=-0.0285 0.0764999999999998 0.000240733268207556 rpy=0 0 1.5707963267949
- joint joint9: axis 0 0 -1 -> 0 0 1; limit lower=-0.6 upper=0.6 effort=10 velocity=6.2 -> lower=-1 upper=1 effort=5 velocity=3.2; origin xyz=0.0515 -0.0119999999999994 0 rpy=-1.5707963267949 0 0 -> xyz=0.0300000000000002 0 0 rpy=1.5707963267949 0 0
